File: audio/audio.kicad_pcb (KiCad board)
At the start: 2 copper layers, 52 x 26 mm, 72 parts, among them P1 CONN_02X01, P2 CONN_01X04, P3 CONN_02X01, P4 CONN_02X01, U1 PCM2912A, U2 MIC, U3 FB, U4 FB, U5 NAU8223, U6 FB, U7 FB, X1 6MHz

Commit message: changed mic. board done...i hope
Parts:
- removed 1PIN, 2PIN, 3PIN, 4PIN: P***, Connect:1pin
- removed C33: 10uF, SMD_Packages:SMD-0603
- removed the G*** at (150.8, 104.1)
- removed JP5: GS0, Connect:GS2
- removed P4: CONN_02X01, Pin_Headers:Pin_Header_Straight_2x01
- added D3: GREEN, LEDs:LED-0603, F.Cu at (158.1, 115.3)
- added G***: LOGO, MIC:logo, B.Cu at (150.8, 104.1)
- added PIN1: PIN1, Connect:1pin, F.Cu at (173.8, 114.1)
- added PIN2: PIN1, Connect:1pin, F.Cu at (173.8, 94.1)
- added PIN3: PIN1, Connect:1pin, F.Cu at (127.8, 114.1)
- added PIN4: PIN1, Connect:1pin, F.Cu at (127.8, 94.1)
- C10: value 0.47uF -> 2.2uF
- C17: value 1uF -> 0.1uF
- C18, C26, C32: value 0.1uF -> 10uF
- C19: value 10uF -> 1nF
- C20, C22, C29: value 1nF -> 0.47uF
- C21, C28, C30: value 0.47uF -> 1nF
- C23: value 0.47uF -> 10uF
- C24: value 10uF -> 0.1uF
- C27: value 10uF -> 0.47uF
- C31: value 1nF -> 0.1uF
- C8: value 1uF -> 22pF
- C9: value 22pF -> 0.1uF
- JP1: value HGAIN -> JUMPER
- JP2: value LGAIN -> JUMPER
- JP3: value XMIC -> HGS
- JP4: value GS5 -> LGS
- R11: value 4K7 -> 510R; moved to F.Cu
- moved R11 22.3 mm to (160.8, 115.3), turned to 270 degrees
- moved C27 22.3 mm to (161.9, 94.1)
- moved R4 20.3 mm to (145.5, 94.1), turned to 180 degrees
- moved C10 20.3 mm to (149.6, 112.6), turned to 180 degrees
- moved P1 17.5 mm to (152.1, 115.6)
- moved C22 17.3 mm to (158.1, 112.6)
- moved R3 16.6 mm to (157.9, 94.1)
- moved P2 14.4 mm to (140.2, 115.7)
- moved C29 13.7 mm to (153.8, 97.2)
- moved C23 11.9 mm to (165.7, 97.2)
- moved JP3 10.2 mm to (149.9, 93.5)
- moved JP2 9.67 mm to (160.0, 93.5), turned to 90 degrees
- moved JP1 9.67 mm to (156.7, 93.5)
- moved C28 9.04 mm to (162.4, 110.1)
- moved C11 8.84 mm to (137.8, 102.4), turned to 180 degrees
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Connections:
- C10 pad 2: Net-(C10-Pad2) -> XOUT
- C19 pad 1: +5VA -> Net-(C19-Pad1)
- C20 pad 2: XGND -> R_IN
- C21 pad 2: R_IN -> XGND
- C23 pad 1: Net-(C23-Pad1) -> +5VA
- C27 pad 1: +5VA -> Net-(C27-Pad1)
- C29 pad 1: Net-(C29-Pad1) -> L_IN
- C29 pad 2: XGND -> Net-(C29-Pad2)
- C30 pad 1: L_IN -> Net-(C30-Pad1)
- C30 pad 2: Net-(C30-Pad2) -> XGND
- C31 pad 1: Net-(C31-Pad1) -> +5VA
- C8 pad 1: XOUT -> Net-(C8-Pad1)
- C8 pad 2: Net-(C8-Pad2) -> XGND
- C9 pad 1: Net-(C9-Pad1) -> XPWR
- JP1 pad 1: XGAIN -> XPWR
- JP1 pad 2: +5VA -> Net-(JP1-Pad2)
- JP2 pad 1: XGAIN -> XOUT
- JP2 pad 2: XGND -> Net-(JP2-Pad2)
- JP3 pad 1: Net-(JP3-Pad1) -> +5VA
- JP3 pad 2: +5VA -> Net-(JP3-Pad2)
- JP4 pad 1: +5VA -> XGND
- JP4 pad 2: Net-(JP4-Pad2) -> Net-(JP3-Pad2)
- P2 pad 1: +5VA -> XPWR
- P2 pad 3: XGAIN -> XOUT
- P2 pad 4: XOUT -> EN
- P3 pad 1: EN -> +5VA
- R10 pad 2: Net-(C9-Pad1) -> Net-(C8-Pad1)
- R11 pad 1: XGND -> Net-(D3-Pad1)
- R11 pad 2: Net-(C10-Pad1) -> +5VA
- SP1 pad 1: Net-(C20-Pad1) -> Net-(C19-Pad1)
- SP1 pad 2: Net-(C22-Pad1) -> Net-(C21-Pad1)
- SP2 pad 1: Net-(C31-Pad1) -> Net-(C30-Pad1)
- SP2 pad 2: Net-(C29-Pad1) -> Net-(C28-Pad1)
- U1 pad 16: Net-(C8-Pad2) -> Net-(C10-Pad1)
- U1 pad 17: Net-(U1-Pad17) -> XPWR
- U1 pad 7: Net-(C9-Pad1) -> Net-(C8-Pad1)
- U2 pad 1: XOUT -> Net-(JP2-Pad2)
- U2 pad 2: XGAIN -> XGND
- U2 pad 3: Net-(C10-Pad2) -> Net-(JP1-Pad2)
- U3 pad 1: Net-(C20-Pad1) -> Net-(C19-Pad1)
- U4 pad 1: Net-(C22-Pad1) -> Net-(C21-Pad1)
- U5 pad 10: Net-(C28-Pad1) -> Net-(C27-Pad1)
- U5 pad 11: Net-(C30-Pad2) -> Net-(C29-Pad2)
- U5 pad 5: Net-(C21-Pad1) -> Net-(C20-Pad1)
- U5 pad 6: Net-(C23-Pad1) -> Net-(C22-Pad1)
- U5 pad 7: Net-(JP4-Pad2) -> Net-(JP3-Pad2)
- U6 pad 1: Net-(C29-Pad1) -> Net-(C28-Pad1)
- U7 pad 1: Net-(C31-Pad1) -> Net-(C30-Pad1)
- USB1 pad 6: (no net) -> XGND
- X1 pad 1: Net-(C9-Pad1) -> Net-(C8-Pad1)
Routing:
- net Net-(C30-Pad1): track 0.00 -> 93.7 mm
- net XOUT: track 106.5 -> 44.9 mm
- net EN: track 40.5 -> 89.6 mm
- net XGAIN: track 46.4 -> 0.00 mm, vias 2 -> 0
- net XPWR: track 0.00 -> 45.0 mm, vias 0 -> 2
- net Net-(C8-Pad1): track 0.00 -> 41.0 mm, vias 0 -> 1
- net +5VA: track 170.3 -> 131.6 mm
- net Net-(C19-Pad1): track 0.00 -> 34.8 mm
- net Net-(C9-Pad1): track 34.6 -> 0.00 mm, vias 2 -> 0
- net Net-(C29-Pad1): track 29.5 -> 0.00 mm
- net Net-(C30-Pad2): track 23.9 -> 0.00 mm, vias 1 -> 0
- net Net-(C2-Pad2): track 40.6 -> 17.4 mm
- net Net-(C31-Pad1): track 23.1 -> 0.00 mm
- net Net-(C27-Pad1): track 0.00 -> 19.5 mm, vias 0 -> 1
- net Net-(P1-Pad2): track 38.5 -> 20.9 mm
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Other:
- net class Default: via_dia 0.635 -> 0.7366
- net class normal: via_dia 0.635 -> 0.7366
- rule pad_to_mask_clearance: 0 -> 0.0508
- rule via_min_size: 0.635 -> 0.7366
- board text added: "EN OUT - +"
- board text removed: "EN -"
- board text removed: "HGN"
- board text removed: "LGN"
- board text removed: "OUT GN - +"

Commit message: board is ready
Parts:
- added G***: LOGO, MIC:OSLOGO, F.Cu at (150.1, 110.1)
Other:
- net class power: via_dia 0.889 -> 0.9906
